Commit message: Update F450 configuration and URDF parameters; adjust mass, inertia, and dimensions for improved accuracy

File: resources/robots/f450/model.urdf (robot description, URDF)
Before this commit: robot f450, 5 links, 4 joints
Links:
- link back_left_prop: mass 0.013 -> 0.014; geometry visual cylinder length=0.01 radius=0.127
- link back_right_prop: mass 0.013 -> 0.014; geometry visual cylinder length=0.01 radius=0.127
- link base_link: mass 1.947 -> 2.317; geometry collision box size=0.57927 0.57927 0.211577; visual box size=0.18 0.18 0.08
- link front_left_prop: mass 0.013 -> 0.014; geometry visual cylinder length=0.01 radius=0.127
- link front_right_prop: mass 0.013 -> 0.014; geometry visual cylinder length=0.01 radius=0.127
